File: PCB/_autosave-rc.kicad_sch (KiCad schematic)
At the start: 21 parts, among them J1 Conn_01x03_Pin, J10 Conn_01x03_Pin, J11 Conn_01x03_Pin, J12 USB4120-03-C_REVA, J2 Conn_01x03_Pin, J3 Conn_01x03_Pin, J4 Conn_01x03_Pin, J5 Conn_01x03_Pin, J6 Conn_01x03_Pin, J7 Conn_01x03_Pin, J8 Conn_01x03_Pin, J9 Conn_01x03_Pin, SW1 SW_Push, U1 ME6211C33M5, U2 ESP32-S3-MINI-1U

Commit message: diodes
Parts:
- added D2, D3: D, Diode_SMD:D_0603_1608Metric_Pad1.05x0.95mm_HandSolder, symbol Device:D
- added U3: ESP32-C6-MINI-1/U, PCM_Espressif:ESP32-C6-MINI-1, symbol PCM_Espressif:ESP32-C6-MINI-1/U
Connections:
- net at J1.2 (Pin_2), J10.2 (Pin_2), J11.2 (Pin_2)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: now also D3.2 (A)
- net at C2.1, U1.1 (V_{IN}), U1.3 (CE): now also D2.1 (K), D3.1 (K)
- net at J12.A4 (VBUS_A): now also J12.A9 (VBUS_A__1), J12.B4 (VBUS_B), J12.B9 (VBUS_B__1), D2.2 (A)
- new net: U3.1 (GND), U3.11 (GND), U3.14 (GND), U3.2 (GND), U3.36 (GND), U3.37 (GND), U3.38 (GND), U3.39 (GND), U3.40 (GND), U3.41 (GND), U3.42 (GND), U3.43 (GND), U3.44 (GND), U3.45 (GND), U3.46 (GND), U3.47 (GND), U3.48 (GND), U3.49 (GND), U3.50 (GND), U3.51 (GND), U3.52 (GND), U3.53 (GND)
