File: PCB/rc.kicad_pcb (KiCad board)
At the start: 2 copper layers, 31.8 x 19 mm, 13 parts, among them J1 Conn_01x03_Pin, J10 Conn_01x03_Pin, J11 Conn_01x03_Pin, J2 Conn_01x03_Pin, J3 Conn_01x03_Pin, J4 Conn_01x03_Pin, J5 Conn_01x03_Pin, J6 Conn_01x03_Pin, J7 Conn_01x03_Pin, J8 Conn_01x03_Pin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

Commit message: smaller
Parts:
- U2: moved to B.Cu
- moved P1 9.91 mm to (38.7, 129.5), turned to 180 degrees
- moved J10 8.86 mm to (44.5, 123.9)
- moved J11 8.86 mm to (47.0, 123.9)
- moved J8 8.40 mm to (44.5, 132.2)
- moved J9 8.40 mm to (47.0, 132.2)
- moved U2 1.03 mm to (34.0, 129.3), turned to -90 degrees
Routing:
- net Net-(J5-Pin_1): track 26.8 -> 11.7 mm
- net Net-(J6-Pin_1): track 25.8 -> 12.2 mm
- net Net-(J4-Pin_1): track 26.7 -> 13.5 mm, vias 1 -> 0
- net Net-(J10-Pin_1): track 17.5 -> 6.49 mm
- net Net-(J3-Pin_1): track 24.7 -> 14.4 mm, vias 1 -> 0
- net Net-(J11-Pin_1): track 20.7 -> 11.3 mm
- net Net-(J1-Pin_1): track 22.2 -> 31.2 mm
- net Net-(J7-Pin_1): track 24.8 -> 19.4 mm
- net Net-(J2-Pin_1): track 19.7 -> 14.4 mm, vias 1 -> 0
- net Net-(J1-Pin_2): track 39.1 -> 34.5 mm
- net Net-(P1-VBUS-PadA4): track 9.08 -> 5.08 mm
- net Net-(J8-Pin_1): track 19.9 -> 22.0 mm
- net Net-(P1-D-): track 2.06 -> 3.82 mm, vias 0 -> 1
- net Net-(P1-D+): track 2.04 -> 3.68 mm, vias 0 -> 1
- net Net-(J9-Pin_1): track 22.8 -> 24.2 mm
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Other:
- board size 31.8 x 19 mm -> 31.1 x 17.8 mm

Commit message: more components
Parts:
- removed P1: USB_C_Plug_USB2.0, Connector_USB:USB_C_Plug_ShenzhenJingTuoJin_918-118A2021Y40002_Vertical
- added C1: C, Capacitor_SMD:C_0402_1005Metric_Pad0.74x0.62mm_HandSolder, F.Cu at (39.4, 127.2)
- added C2: C, Capacitor_SMD:C_0402_1005Metric_Pad0.74x0.62mm_HandSolder, F.Cu at (37.5, 127.3)
- added D1: LED, LED_THT:LED_D3.0mm, F.Cu at (36.2, 137.8)
- added J12: USB4120-03-C_REVA, usbc:USB4120-03-C_GCT, F.Cu at (29.6, 137.7)
- added R1: R_US, Resistor_SMD:R_0402_1005Metric_Pad0.72x0.64mm_HandSolder, F.Cu at (34.9, 133.3)
- added R2: R_US, Resistor_SMD:R_0402_1005Metric_Pad0.72x0.64mm_HandSolder, F.Cu at (31.1, 128.2)
- added R3: R_US, Resistor_SMD:R_0402_1005Metric_Pad0.72x0.64mm_HandSolder, B.Cu at (41.9, 137.8)
- added SW1: SW_Push, Button_Switch_SMD:SW_Tactile_SPST_NO_Straight_CK_PTS636Sx25SMTRLFS, F.Cu at (32.4, 123.2)
- added U1: ME6211C33M5, Package_TO_SOT_SMD:SOT-23-5, F.Cu at (38.7, 131.1)
- moved J1 0.38 mm to (50.8, 137.4)
- moved J2 0.38 mm to (50.8, 134.9)
- moved J3 0.38 mm to (50.8, 132.4)
- moved J4 0.38 mm to (50.8, 129.9)
- moved J10 0.38 mm to (44.5, 123.5)
- moved J11 0.38 mm to (47.0, 123.5)
- moved J5 0.38 mm to (50.8, 127.4)
- moved J6 0.38 mm to (50.8, 124.9)
- moved J7 0.38 mm to (50.8, 122.4)
- moved J8 0.38 mm to (44.5, 131.8)
- moved J9 0.38 mm to (47.0, 131.8)
- moved U2 0.38 mm to (34.0, 128.9)
Connections:
- U2 pad 3: unconnected-(U2-3V3-Pad3) -> Net-(U1-V_{OUT})
- U2 pad 31: unconnected-(U2-IO35-Pad31) -> Net-(U2-IO35)
- U2 pad 9: unconnected-(U2-IO5-Pad9) -> Net-(U2-IO5)
Routing:
- net Net-(D1-K): track 137.0 -> 175.4 mm, vias 1 -> 2
- net Net-(J12-D1-): track 3.82 -> 24.3 mm, vias 1 -> 2
- net Net-(U1-V_{OUT}): track 0.00 -> 18.3 mm, vias 0 -> 1
- net Net-(J12-D1+): track 3.68 -> 16.7 mm
- net Net-(J1-Pin_1): track 31.2 -> 18.7 mm
- net Net-(J12-CC1): track 0.00 -> 10.3 mm
- net Net-(U1-CE): track 0.00 -> 5.19 mm
- net Net-(P1-VBUS-PadA4): track 5.08 -> 0.00 mm
- net Net-(D1-A): track 0.00 -> 4.27 mm
- net Net-(J12-CC2): track 0.00 -> 3.92 mm
- net Net-(U2-IO5): track 0.00 -> 3.82 mm, vias 0 -> 1
- net Net-(J3-Pin_1): track 14.4 -> 17.4 mm
- net Net-(U2-IO35): track 0.00 -> 2.58 mm
- net Net-(J8-Pin_1): track 22.0 -> 19.8 mm
- net Net-(J2-Pin_1): track 14.4 -> 15.9 mm
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Other:
- board size 31.1 x 17.8 mm -> 32.4 x 19 mm

Commit message: diodes
Parts:
- added D2: D, Diode_SMD:D_0603_1608Metric_Pad1.05x0.95mm_HandSolder, F.Cu at (38.1, 134.6)
- added D3: D, Diode_SMD:D_0603_1608Metric_Pad1.05x0.95mm_HandSolder, B.Cu at (43.8, 139.1)
- added U3: ESP32-C6-MINI-1/U, PCM_Espressif:ESP32-C6-MINI-1, F.Cu at (66.4, 128.9)
- R3: moved to F.Cu
- moved D1 2.55 mm to (38.7, 137.8), turned to 180 degrees
- moved C2 1.02 mm to (37.5, 128.3), turned to 180 degrees
- moved R3 0.63 mm to (41.3, 137.8), turned to 0 degrees
- moved C1 0.39 mm to (39.4, 127.6), turned to -90 degrees
Connections:
- J12 pad A4: unconnected-(J12-VBUS_A-PadA4) -> Net-(D2-A)
- J12 pad A9: unconnected-(J12-VBUS_A__1-PadA9) -> Net-(D2-A)
- J12 pad B4: unconnected-(J12-VBUS_B-PadB4) -> Net-(D2-A)
- J12 pad B9: unconnected-(J12-VBUS_B__1-PadB9) -> Net-(D2-A)
Routing:
- net Net-(D2-A): track 0.00 -> 22.8 mm
- net Net-(D2-K): track 5.19 -> 17.2 mm, vias 0 -> 2
- net Net-(D3-A): track 34.0 -> 39.6 mm, vias 0 -> 1
- net Net-(J12-CC1): track 10.3 -> 13.8 mm
- net Net-(J3-Pin_1): track 17.4 -> 14.4 mm
- net Net-(U1-V_{OUT}): track 18.3 -> 21.1 mm
- net Net-(J12-D1-): track 24.3 -> 22.8 mm
- net Net-(D1-A): track 4.27 -> 5.80 mm
- net Net-(U2-IO35): track 2.58 -> 3.65 mm, vias 0 -> 1
- net Net-(D1-K): track 175.4 -> 174.5 mm, vias 2 -> 3
- net Net-(J12-D1+): track 16.7 -> 16.0 mm
- net Net-(J8-Pin_1): track 19.8 -> 20.4 mm

Commit message: c6
Parts:
- removed U2: ESP32-S3-MINI-1U, RF_Module:ESP32-S2-MINI-1U
- D3: moved to F.Cu
- R1, R2, R3: moved to B.Cu
- U3: footprint PCM_Espressif:ESP32-C6-MINI-1 -> PCM_Espressif:ESP32-C3-MINI-1_HandSoldering; moved to B.Cu
- moved U3 33.7 mm to (33.0, 132.7)
- moved J12 15.0 mm to (29.4, 122.6), turned to 0 degrees
- moved D1 14.8 mm to (41.3, 123.2)
- moved R3 13.3 mm to (37.5, 125.1), turned to 180 degrees
- moved C1 11.7 mm to (29.2, 133.3)
- moved U1 10.8 mm to (27.9, 130.2)
- moved C2 10.8 mm to (27.9, 133.3), turned to -90 degrees
- moved R1 10.3 mm to (36.8, 123.2)
- moved D3 9.53 mm to (36.2, 133.3), turned to -90 degrees
- moved D2 8.64 mm to (31.1, 129.5), turned to 90 degrees
- moved SW1 8.13 mm to (37.5, 129.5)
- moved R2 6.72 mm to (26.7, 123.2), turned to 90 degrees
- moved J8 0.64 mm to (44.5, 132.4)
- moved J9 0.64 mm to (47.0, 132.4)
Connections:
- R3 pad 2: Net-(U2-IO35) -> Net-(U3-GPIO8)
- SW1 pad 2: Net-(U2-IO5) -> Net-(U3-GPIO15)
- U3 pad 1: Net-(U3-GND-Pad1) -> Net-(D1-K)
- U3 pad 11: Net-(U3-GND-Pad1) -> Net-(D1-K)
- U3 pad 14: Net-(U3-GND-Pad1) -> Net-(D1-K)
- U3 pad 17: unconnected-(U3-GPIO12/USB_D--Pad17) -> Net-(J12-D1-)
- U3 pad 18: unconnected-(U3-GPIO13/USB_D+-Pad18) -> Net-(J12-D1+)
- U3 pad 2: Net-(U3-GND-Pad1) -> Net-(D1-K)
- U3 pad 20: unconnected-(U3-GPIO15-Pad20) -> Net-(U3-GPIO15)
- U3 pad 22: unconnected-(U3-GPIO8-Pad22) -> Net-(U3-GPIO8)
- U3 pad 23: unconnected-(U3-GPIO9-Pad23) -> Net-(J7-Pin_1)
- U3 pad 24: unconnected-(U3-GPIO18-Pad24) -> Net-(J11-Pin_1)
- U3 pad 25: unconnected-(U3-GPIO19-Pad25) -> Net-(J10-Pin_1)
- U3 pad 26: unconnected-(U3-GPIO20-Pad26) -> Net-(J6-Pin_1)
- U3 pad 27: unconnected-(U3-GPIO21-Pad27) -> Net-(J5-Pin_1)
- U3 pad 28: unconnected-(U3-GPIO22-Pad28) -> Net-(J4-Pin_1)
- U3 pad 29: unconnected-(U3-GPIO23-Pad29) -> Net-(J9-Pin_1)
- U3 pad 3: unconnected-(U3-3V3-Pad3) -> Net-(U1-V_{OUT})
- U3 pad 30: unconnected-(U3-U0RXD/GPIO17-Pad30) -> Net-(J8-Pin_1)
- U3 pad 31: unconnected-(U3-U0TXD/GPIO16-Pad31) -> Net-(J3-Pin_1)
- U3 pad 36: Net-(U3-GND-Pad1) -> Net-(D1-K)
- U3 pad 37: Net-(U3-GND-Pad1) -> Net-(D1-K)
- U3 pad 38: Net-(U3-GND-Pad1) -> Net-(D1-K)
- U3 pad 39: Net-(U3-GND-Pad1) -> Net-(D1-K)
- U3 pad 40: Net-(U3-GND-Pad1) -> Net-(D1-K)
- U3 pad 41: Net-(U3-GND-Pad1) -> Net-(D1-K)
- U3 pad 42: Net-(U3-GND-Pad1) -> Net-(D1-K)
- U3 pad 43: Net-(U3-GND-Pad1) -> Net-(D1-K)
- U3 pad 44: Net-(U3-GND-Pad1) -> Net-(D1-K)
- U3 pad 45: Net-(U3-GND-Pad1) -> Net-(D1-K)
- U3 pad 46: Net-(U3-GND-Pad1) -> Net-(D1-K)
- U3 pad 47: Net-(U3-GND-Pad1) -> Net-(D1-K)
- U3 pad 48: Net-(U3-GND-Pad1) -> Net-(D1-K)
- U3 pad 49: Net-(U3-GND-Pad1) -> Net-(D1-K)
- U3 pad 5: unconnected-(U3-GPIO2/ADC1_CH2-Pad5) -> Net-(J1-Pin_1)
- U3 pad 50: Net-(U3-GND-Pad1) -> Net-(D1-K)
- U3 pad 51: Net-(U3-GND-Pad1) -> Net-(D1-K)
- U3 pad 52: Net-(U3-GND-Pad1) -> Net-(D1-K)
- U3 pad 53: Net-(U3-GND-Pad1) -> Net-(D1-K)
- U3 pad 6: unconnected-(U3-GPIO3/ADC1_CH3-Pad6) -> Net-(J2-Pin_1)
Routing:
- net Net-(D1-K): track 174.5 -> 152.0 mm, vias 3 -> 1
- net Net-(J8-Pin_1): track 20.4 -> 5.22 mm, vias 1 -> 0
- net Net-(J9-Pin_1): track 23.6 -> 8.72 mm, vias 1 -> 0
- net Net-(J2-Pin_1): track 15.9 -> 30.7 mm, vias 0 -> 1
- net Net-(J12-D1-): track 22.8 -> 8.46 mm
- net Net-(U1-V_{OUT}): track 21.1 -> 7.30 mm
- net Net-(J1-Pin_1): track 18.5 -> 30.0 mm
- net Net-(J12-D1+): track 16.0 -> 5.18 mm
- net Net-(U3-GPIO15): track 0.00 -> 8.24 mm, vias 0 -> 1
- net Net-(J12-CC1): track 13.8 -> 6.48 mm, vias 0 -> 1
- net Net-(D2-A): track 22.8 -> 17.2 mm, vias 0 -> 2
- net Net-(D3-A): track 39.6 -> 43.6 mm, vias 1 -> 0
- net Net-(U2-IO5): track 3.82 -> 0.00 mm, vias 1 -> 0
- net Net-(U2-IO35): track 3.65 -> 0.00 mm, vias 1 -> 0
- net Net-(D1-A): track 5.80 -> 2.19 mm
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Other:
- board size 32.4 x 19 mm -> 33 x 19 mm
