File: PCB/rc.kicad_sch (KiCad schematic)
At the start: 13 parts, among them J1 Conn_01x03_Pin, J10 Conn_01x03_Pin, J11 Conn_01x03_Pin, J2 Conn_01x03_Pin, J3 Conn_01x03_Pin, J4 Conn_01x03_Pin, J5 Conn_01x03_Pin, J6 Conn_01x03_Pin, J7 Conn_01x03_Pin, J8 Conn_01x03_Pin, J9 Conn_01x03_Pin, P1 USB_C_Plug_USB2.0, U2 ESP32-S3-MINI-1U

Commit message: more components
Parts:
- removed P1: USB_C_Plug_USB2.0, Connector_USB:USB_C_Plug_ShenzhenJingTuoJin_918-118A2021Y40002_Vertical, symbol Connector:USB_C_Plug_USB2.0
- added C1, C2: C, Capacitor_SMD:C_0402_1005Metric_Pad0.74x0.62mm_HandSolder, symbol Device:C
- added D1: LED, LED_THT:LED_D3.0mm, symbol Device:LED
- added J12: USB4120-03-C_REVA, usbc:USB4120-03-C_GCT, symbol usbc:USB4120-03-C_REVA
- added R1, R2: R_US, Resistor_SMD:R_0402_1005Metric_Pad0.72x0.64mm_HandSolder, symbol Device:R_US
- added SW1: SW_Push, Button_Switch_SMD:SW_Tactile_SPST_NO_Straight_CK_PTS636Sx25SMTRLFS, symbol Switch:SW_Push
- added U1: ME6211C33M5, Package_TO_SOT_SMD:SOT-23-5, symbol Regulator_Linear:ME6211C33M5
Connections:
- net at J1.3 (Pin_3), J10.3 (Pin_3), J11.3 (Pin_3)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: now also C1.2, C2.2, D1.1 (K), J12.A1 (GND_A), J12.A12 (GND_A__1), J12.B1 (GND_B), J12.B12 (GND_B__1), J12.S1 (SHIELD), J12.S2 (SHIELD__1), J12.S3 (SHIELD__2), J12.S4 (SHIELD__3), R1.1, R2.1, SW1.1, U1.2 (V_{SS})
- net at U2.23 (IO19): now also J12.A7 (D1-), J12.B7 (D2-)
- net at U2.24 (IO20): now also J12.A6 (D1+), J12.B6 (D2+)
- net at U2.3 (3V3): now also C1.1, U1.5 (V_{OUT})
- net at U2.31 (IO35): now also D1.2 (A)
- net at U2.9 (IO5): now also SW1.2
- new net: J12.B5 (CC2), R1.2
- new net: J12.A5 (CC1), R2.2
- new net: C2.1, U1.1 (V_{IN}), U1.3 (CE)

Commit message: diodes
Parts:
- added D2, D3: D, Diode_SMD:D_2010_5025Metric_Pad1.52x2.65mm_HandSolder, symbol Device:D
- added R3: R_US, Resistor_SMD:R_0402_1005Metric_Pad0.72x0.64mm_HandSolder, symbol Device:R_US
- added U3: ESP32-C6-MINI-1/U, PCM_Espressif:ESP32-C6-MINI-1, symbol PCM_Espressif:ESP32-C6-MINI-1/U
Connections:
- net at J1.2 (Pin_2), J10.2 (Pin_2), J11.2 (Pin_2)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: now also D3.2 (A)
- net at C2.1, U1.1 (V_{IN}), U1.3 (CE): now also D2.1 (K), D3.1 (K)
- net at J12.A4 (VBUS_A): now also J12.A9 (VBUS_A__1), J12.B4 (VBUS_B), J12.B9 (VBUS_B__1), D2.2 (A)
- net at D1.2 (A): now also R3.1; no longer U2.31 (IO35)
- new net: U3.1 (GND), U3.11 (GND), U3.14 (GND), U3.2 (GND), U3.36 (GND), U3.37 (GND), U3.38 (GND), U3.39 (GND), U3.40 (GND), U3.41 (GND), U3.42 (GND), U3.43 (GND), U3.44 (GND), U3.45 (GND), U3.46 (GND), U3.47 (GND), U3.48 (GND), U3.49 (GND), U3.50 (GND), U3.51 (GND), U3.52 (GND), U3.53 (GND)
- new net: R3.2, U2.31 (IO35)

Commit message: c6
Parts:
- removed U2: ESP32-S3-MINI-1U, RF_Module:ESP32-S2-MINI-1U, symbol RF_Module:ESP32-S3-MINI-1U
- D2, D3: footprint Diode_SMD:D_2010_5025Metric_Pad1.52x2.65mm_HandSolder -> Diode_SMD:D_0603_1608Metric_Pad1.05x0.95mm_HandSolder
- U3: footprint PCM_Espressif:ESP32-C6-MINI-1 -> PCM_Espressif:ESP32-C3-MINI-1_HandSoldering
Connections:
- net at U3.1 (GND), U3.11 (GND), U3.14 (GND)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: now also C1.2, C2.2, D1.1 (K), J1.3 (Pin_3), J10.3 (Pin_3), J11.3 (Pin_3), J12.A1 (GND_A), J12.A12 (GND_A__1), J12.B1 (GND_B), J12.B12 (GND_B__1), J12.S1 (SHIELD), J12.S2 (SHIELD__1), J12.S3 (SHIELD__2), J12.S4 (SHIELD__3), J2.3 (Pin_3), J3.3 (Pin_3), J4.3 (Pin_3), J5.3 (Pin_3), J6.3 (Pin_3), J7.3 (Pin_3), J8.3 (Pin_3), J9.3 (Pin_3), R1.1, R2.1, SW1.1, U1.2 (V_{SS})
- net at U3.17 (GPIO12/USB_D-): now also J12.A7 (D1-), J12.B7 (D2-)
- net at U3.18 (GPIO13/USB_D+): now also J12.A6 (D1+), J12.B6 (D2+)
- net at U3.20 (GPIO15): now also SW1.2
- net at U3.22 (GPIO8): now also R3.2
- net at U3.23 (GPIO9): now also J7.1 (Pin_1)
- net at U3.24 (GPIO18): now also J11.1 (Pin_1)
- net at U3.25 (GPIO19): now also J10.1 (Pin_1)
- net at U3.26 (GPIO20): now also J6.1 (Pin_1)
- net at U3.27 (GPIO21): now also J5.1 (Pin_1)
- net at U3.28 (GPIO22): now also J4.1 (Pin_1)
- net at U3.29 (GPIO23): now also J9.1 (Pin_1)
- net at U3.3 (3V3): now also C1.1, U1.5 (V_{OUT})
- net at U3.30 (U0RXD/GPIO17): now also J8.1 (Pin_1)
- net at U3.31 (U0TXD/GPIO16): now also J3.1 (Pin_1)
- net at U3.5 (GPIO2/ADC1_CH2): now also J1.1 (Pin_1)
- net at U3.6 (GPIO3/ADC1_CH3): now also J2.1 (Pin_1)
Other:
- moved on the sheet: U3
